Commit message: add view robot launch

File: src/bob_description/urdf/diffbot.urdf.xacro (robot description, xacro)
@@ -1,15 +1,14 @@
 <?xml version="1.0"?>
-<robot xmlns:xacro="http://www.ros.org/wiki/xacro"  name="robot">
-^   <xacro:arg name="prefix" default="" />
-    <xacro:arg name="use_mock_hardware" default="false" />
-    <xacro:include filename="$(find bob_description)/urdf/robot_core.xacro" />
-    <xacro:include filename="$(find bob_description)/urdf/robot.gazebo" />
-    <xacro:include filename="$(find bob_description)/urdf/lidar.xacro" />
-    <xacro:include filename="$(find bob_description)/urdf/camera.xacro" />
-    <xacro:include filename="$(find bob_description)/urdf/accelerometer.xacro" />
-    <!-- Import diffbot ros2_control description -->
-    <xacro:include filename="$(find bob_description)/ros2_control/diffbot.ros2_control.xacro" />
-    <xacro:diffbot prefix="$(arg prefix)" />
-    <xacro:diffbot_ros2_control
-        name="DiffBot" prefix="$(arg prefix)" use_mock_hardware="$(arg use_mock_hardware)"/>
+<!-- Basic differential drive mobile base -->
+<robot xmlns:xacro="http://www.ros.org/wiki/xacro" name="diffdrive_robot">
+  <xacro:arg name="prefix" default="" />
+  <xacro:arg name="use_mock_hardware" default="false" />
+  <xacro:include filename="$(find bob_description)/urdf/diffbot_description.urdf.xacro" />
+  <!-- Import Rviz colors -->
+  <xacro:include filename="$(find bob_description)/urdf/diffbot.materials.xacro" />
+  <!-- Import diffbot ros2_control description -->
+  <xacro:include filename="$(find bob_description)/ros2_control/diffbot.ros2_control.xacro" />
+  <xacro:diffbot prefix="$(arg prefix)" />
+  <xacro:diffbot_ros2_control
+    name="DiffBot" prefix="$(arg prefix)" use_mock_hardware="$(arg use_mock_hardware)"/>
 </robot>

File: src/bob_description/urdf/robot_core.xacro (robot description, xacro)
@@ -1,4 +1,5 @@
 <?xml version="1.0"?>
 <robot xmlns:xacro="http://www.ros.org/wiki/xacro" >
+    <xacro:macro name="diffbot" params="prefix">
     <!-- Body Dimensions -->
     <xacro:property name="main_body_x_dim" value="0.4"/>
