Commit message: added gazebo launch

File: src/bob_description/urdf/robot_core.xacro (robot description, xacro)
@@ -1,5 +1,4 @@
 <?xml version="1.0"?>
 <robot xmlns:xacro="http://www.ros.org/wiki/xacro" >
-    <xacro:macro name="diffbot" params="prefix">
     <!-- Body Dimensions -->
     <xacro:property name="main_body_x_dim" value="0.4"/>

Commit message: printing to terminal

File: src/bob_description/urdf/robot_core.xacro (robot description, xacro)
@@ -21,5 +21,5 @@
     <!-- Rear Wheel Dimensions -->
     <xacro:property name="wheel_link_radius" value="0.08255"/>
-    <xacro:property name="wheel_link_length" value="0.037"/>
+    <xacro:property name="wheel_link_length" value="0.068"/>
     <xacro:property name="wheel_link_z_location" value="0"/>
     <!-- Front Wheel Dimensions -->
