Commit message: added slam

File: src/bob_description/urdf/bob_core.xacro (robot description, xacro)
@@ -77,4 +77,11 @@
     <link name="base_link">
     </link>
+    <joint name="base_footprint_joint" type="fixed">
+        <parent link="base_link"/>front_
+        <child link="base_footprint"/>front_
+        <origin xyz="0 0 0" rpy="0 0 0"/>
+    </joint>
+    <link name="base_footprint">
+    </link>
     <!-- CHASSIS LINK -->
     <joint name="chassis_joint" type="fixed">

Commit message: changed frames

File: src/bob_description/urdf/bob_core.xacro (robot description, xacro)
@@ -27,5 +27,5 @@
     <xacro:property name="front_wheel_link_length" value="0.015"/>
     <xacro:property name="front_wheel_link_x_offset" value="0.075"/>
-    <xacro:property name="front_wheel_link_x_location" value="${main_body_x_dim+front_wheel_mount_x_dim-front_wheel_link_x_offset}"/>
+    <xacro:property name="front_wheel_link_x_location" value="${main_body_x_dim+front_wheel_mount_x_dim-wheel_link_radius-front_wheel_link_x_offset}"/>
     <!-- Material Density -->
     <xacro:property name="body_density" value="2710.0"/>
@@ -75,12 +75,11 @@
     </xacro:macro>
     <!-- BASE LINK -->
-    <link name="base_link">
-    </link>
-    <joint name="base_footprint_joint" type="fixed">
-        <parent link="base_link"/>front_
-        <child link="base_footprint"/>front_
+   <link name="base_footprint"/>
+    <joint name="base_joint" type="fixed">
+        <parent link="base_footprint"/>front_
+        <child link="base_link"/>front_
         <origin xyz="0 0 0" rpy="0 0 0"/>
     </joint>
-    <link name="base_footprint">
+     <link name="base_link">
     </link>
     <!-- CHASSIS LINK -->
@@ -275,5 +274,5 @@
     <!-- CASTER WHEEL LINK -->
     <joint name="caster_wheel_joint" type="fixed">
-        <parent link="wheel_mount"/>
+        <parent link="base_link"/>
         <child link="caster_wheel"/>
         <origin xyz="${front_wheel_link_x_location} 0 ${(main_body_z_dim-front_wheel_mount_z_dim)-front_wheel_link_radius}"/>

File: src/bob_description/urdf/gazebo_control.xacro (robot description, xacro)
@@ -13,5 +13,5 @@
             <!-- Output -->
             <odometry_frame>odom</odometry_frame>
-            <robot_base_frame>base_link</robot_base_frame>
+            <robot_base_frame>base_footprint</robot_base_frame>
             <publish_odom>true</publish_odom>
             <publish_odom_tf>true</publish_odom_tf>

File: src/bob_description/urdf/imu.xacro (robot description, xacro)
@@ -4,12 +4,13 @@
     <xacro:property name="imu_y_dim" value="0.015"/>
     <xacro:property name="imu_z_dim" value="0.001"/>
-    <xacro:property name="imu_x_offset" value="0.13"/>
+    <xacro:property name="imu_x_offset" value="0.25"/>
+    <xacro:property name="imu_z_offset" value="0.025"/>
     <xacro:property name="imu_density" value="2710.0"/>
     <xacro:property name="imu_mass" value="${imu_density*imu_x_dim*imu_y_dim*imu_z_dim}"/>
     <!-- LIDAR LINK -->
 	<joint name="imu_joint" type="fixed">
-        <parent link="chassis"/>
+        <parent link="base_link"/>
         <child link="imu_frame"/>
-        <origin xyz="${imu_x_offset} 0 ${imu_z_dim*0.5+main_body_z_dim}"/>
+        <origin xyz="${imu_x_offset-wheel_link_radius} 0 ${imu_z_offset}"/>
     </joint>
     <link name="imu_frame">
@@ -35,5 +36,4 @@
             <update_rate>100</update_rate>
             <plugin name="imu_controller" filename="libgazebo_ros_imu_sensor.so">
-                <topic_name>imu</topic_name>
                 <frame_name>imu_frame</frame_name>
                 <ros>
@@ -44,5 +44,5 @@
             <always_on>true</always_on>
             <update_rate>100</update_rate>
-            <visualize>false</visualize>
+            <visualize>true</visualize>
             <imu>
             <angular_velocity>

File: src/bob_description/urdf/lidar.xacro (robot description, xacro)
@@ -9,7 +9,7 @@
     <!-- LIDAR LINK -->
 	<joint name="lidar_joint" type="fixed">
-        <parent link="chassis"/>
+        <parent link="base_link"/>
         <child link="lidar_frame"/>
-        <origin xyz="${lidar_x_location} 0 ${lidar_length*0.5+main_body_z_dim}" rpy="0 0 0"/>
+        <origin xyz="${lidar_x_location-wheel_link_radius} 0 ${lidar_length*0.5+main_body_z_dim}" rpy="0 0 0"/>
     </joint>
     <link name="lidar_frame">
