Commit message: added hardware interfaces

File: src/bob_description/ros2_control/diffbot.ros2_control.xacro (robot description, xacro)
@@ -3,5 +3,4 @@
   <xacro:macro name="diffbot_ros2_control" params="name prefix use_mock_hardware">
     <ros2_control name="${name}" type="system">
-      <xacro:unless value="${use_mock_hardware}">
         <hardware>
           <plugin>bob_base/DiffDriveBobHardware</plugin>
@@ -12,20 +11,17 @@
           <param name="wheel_radius">0.08255</param>
         </hardware>
-      </xacro:unless>
-      <xacro:if value="${use_mock_hardware}">
-        <hardware>
-          <plugin>mock_components/GenericSystem</plugin>
-          <param name="calculate_dynamics">true</param>
-        </hardware>
-      </xacro:if>
-      <joint name="${prefix}left_wheel_joint">
+      <joint name="left_wheel_joint">
         <command_interface name="velocity"/>
         <state_interface name="position"/>
         <state_interface name="velocity"/>
+        <state_interface name="rpm"/>
+        <state_interface name="alarm"/>
       </joint>
-      <joint name="${prefix}right_wheel_joint">
+      <joint name="right_wheel_joint">
         <command_interface name="velocity"/>
         <state_interface name="position"/>
         <state_interface name="velocity"/>
+        <state_interface name="rpm"/>
+        <state_interface name="alarm"/>
       </joint>
     </ros2_control>
