Commit message: added imu code

File: src/bob_description/ros2_control/bob.ros2_control.xacro (robot description, xacro)
@@ -1,8 +1,9 @@
 <?xml version="1.0"?>
 <robot xmlns:xacro="http://www.ros.org/wiki/xacro">
-  <xacro:macro name="diffbot_ros2_control" params="name prefix use_mock_hardware">
-    <ros2_control name="${name}" type="system">
-        <hardware>
-          <plugin>bob_base/DiffDriveBobHardware</plugin>
+  <!-- Real robot ros2_control -->
+  <xacro:unless value="$(arg sim_mode)">
+    <ros2_control name='RealRobot' type='system'>
+      <hardware>
+        <plugin>bob_base/DiffDriveBobHardware</plugin>
           <param name="left_wheel_name">left_wheel_joint</param>
           <param name="right_wheel_name">right_wheel_joint</param>
@@ -10,5 +11,5 @@
           <param name="enc_ticks_per_rev">45</param>
           <param name="wheel_radius">0.08255</param>
-        </hardware>
+      </hardware>
       <joint name="left_wheel_joint">
         <command_interface name="velocity"/>
@@ -26,4 +27,54 @@
       </joint>
     </ros2_control>
-  </xacro:macro>
+    <!-- MPU6050 sensor-->
+    <ros2_control name='MPU6050' type='sensor'>
+      <hardware>
+        <plugin>bob_bringup/MPU6050Hardware</plugin>
+          <param name='sensor_name'>mpu6050</param>
+          <param name='frame_id'>imu_link</param>
+      </hardware>
+      <sensor name='mpu6050'>
+        <state_interface name='orientation.x'/>
+        <state_interface name='orientation.y'/>
+        <state_interface name='orientation.z'/>
+        <state_interface name='orientation.w'/>
+        <state_interface name='angular_velocity.x'/>
+        <state_interface name='angular_velocity.y'/>
+        <state_interface name='angular_velocity.z'/>
+        <state_interface name='linear_acceleration.x'/>
+        <state_interface name='linear_acceleration.y'/>
+        <state_interface name='linear_acceleration.z'/>
+      </sensor>
+    </ros2_control>
+  </xacro:unless>
+  <!-- Gazebo ros2_control -->
+  <xacro:if value="$(arg sim_mode)">
+    <ros2_control name='GazeboSystem' type='system'>
+      <hardware>
+        <plugin>gazebo_ros2_control/GazeboSystem</plugin>
+      </hardware>
+      <joint name='left_wheel_joint'>
+        <command_interface name='velocity'>
+          <param name='min'>-10</param>
+          <param name='max'>10</param>
+        </command_interface>
+        <state_interface name='velocity'/>
+        <state_interface name='position'/>
+      </joint>
+      <joint name='right_wheel_joint'>
+        <command_interface name='velocity'>
+          <param name='min'>-10</param>
+          <param name='max'>10</param>
+        </command_interface>
+        <state_interface name='velocity'/>
+        <state_interface name='position'/>
+      </joint>
+    </ros2_control>
+  </xacro:if>
+  <gazebo>
+    <plugin name='gazebo_ros2_control' filename='libgazebo_ros2_control.so'>
+      <parameters>$(find bob_bringup)/config/bob_controllers.yaml</parameters>
+      <parameters>$(find bob_bringup)/config/gazebo_ros2_ctl_use_sim.yaml</parameters>
+    </plugin>
+  </gazebo>
 </robot>

File: src/bob_description/urdf/bob_core.xacro (robot description, xacro)
@@ -103,4 +103,7 @@
         </inertial>
     </link>
+    <gazebo reference="chassis">
+    <material>Gazebo/White</material>
+    </gazebo>
     <!-- CAMERA MOUNT LINK -->
     <joint name="camera_mount_joint" type="fixed">
@@ -126,4 +129,7 @@
         </inertial>
     </link>
+    <gazebo reference="camera_mount">
+        <material>Gazebo/White</material>
+    </gazebo>
     <!-- EMERGENCY MOUNT LINK -->
     <joint name="emergency_mount_joint" type="fixed">
@@ -149,4 +155,7 @@
         </inertial>
     </link>
+    <gazebo reference="emergency_mount">
+        <material>Gazebo/Black</material>
+    </gazebo>
     <!-- EMERGENCY BUTTON LINK -->
     <joint name="emergency_button_joint" type="fixed">
@@ -172,4 +181,7 @@
         </inertial>
     </link>
+    <gazebo reference="emergency_button">
+        <material>Gazebo/Red</material>
+    </gazebo>
     <!-- WHEEL MOUNT LINK -->
     <joint name="wheel_mount_joint" type="fixed">
@@ -221,4 +233,9 @@
         <xacro:inertia_wheel />
     </link>
+    <gazebo reference="left_wheel">
+    <mu1>0.2</mu1>
+    <mu2>0.2</mu2>
+    <material>Gazebo/Black</material>
+    </gazebo>
     <!-- RIGHT WHEEL LINK -->
     <joint name="right_wheel_joint" type="continuous">
@@ -244,4 +261,9 @@
         <xacro:inertia_wheel />
     </link>
+    <gazebo reference="right_wheel">
+    <mu1>0.2</mu1>
+    <mu2>0.2</mu2>
+    <material>Gazebo/Black</material>
+    </gazebo>
     <!-- CASTER WHEEL LINK -->
     <joint name="caster_wheel_joint" type="fixed">
@@ -264,3 +286,8 @@
         <xacro:inertia_front_wheel />
     </link>
+    <gazebo reference="caster_wheel">
+    <mu1>0.001</mu1>
+    <mu2>0.001</mu2>
+    <material>Gazebo/Black</material>
+    </gazebo>
 </robot>

File: src/bob_description/urdf/camera.xacro (robot description, xacro)
@@ -38,3 +38,26 @@
     </joint>
     <link name="camera_optical_frame"></link>
+    <gazebo reference="camera_frame">
+        <material>Gazebo/Black</material>
+        <sensor name="camera" type="camera">
+            <pose> camera_radius 0 0 0 0 0 </pose>
+            <visualize>true</visualize>
+            <update_rate>10</update_rate>
+            <camera>
+                <horizontal_fov>1.089</horizontal_fov>
+                <image>
+                    <format>R8G8B8</format>
+                    <width>640</width>
+                    <height>480</height>
+                </image>
+                <clip>
+                    <near>0.05</near>
+                    <far>8.0</far>
+                </clip>
+            </camera>
+            <plugin name="camera_controller" filename="libgazebo_ros_camera.so">
+                <frame_name>camera_optical_frame</frame_name>
+            </plugin>
+        </sensor>
+    </gazebo>
 </robot>

File: src/bob_description/urdf/gazebo_control.xacro (robot description, xacro)
@@ -1,34 +1,4 @@
 <?xml version="1.0"?>
 <robot>
-    <gazebo reference="chassis">
-    <material>Gazebo/White</material>
-    </gazebo>
-    <gazebo reference="wheel_mount">
-    <material>Gazebo/White</material>
-    </gazebo>
-    <gazebo reference="camera_mount">
-        <material>Gazebo/White</material>
-    </gazebo>
-    <gazebo reference="emergency_mount">
-        <material>Gazebo/Black</material>
-    </gazebo>
-    <gazebo reference="emergency_button">
-        <material>Gazebo/Red</material>
-    </gazebo>
-    <gazebo reference="left_wheel">
-    <mu1>0.2</mu1>
-    <mu2>0.2</mu2>
-    <material>Gazebo/Black</material>
-    </gazebo>
-    <gazebo reference="right_wheel">
-    <mu1>0.2</mu1>
-    <mu2>0.2</mu2>
-    <material>Gazebo/Black</material>
-    </gazebo>
-    <gazebo reference="caster_wheel">
-    <mu1>0.001</mu1>
-    <mu2>0.001</mu2>
-    <material>Gazebo/Black</material>
-    </gazebo>
     <gazebo>
         <plugin name="diff_drive" filename="libgazebo_ros_diff_drive.so">
@@ -47,149 +17,8 @@
             <publish_odom_tf>true</publish_odom_tf>
             <publish_wheel_tf>true</publish_wheel_tf>
-            <publishWheelJointState>true</publishWheelJointState>
+            <publish_wheel_joint_state>true</publish_wheel_joint_state>
             <command_topic>cmd_vel</command_topic>
             <odometry_topic>odom</odometry_topic>
         </plugin>
     </gazebo>
-    <gazebo reference="lidar_frame">
-        <material>Gazebo/Red</material>
-        <sensor name="lidar" type="ray">
-            <pose> 0 0 0 0 0 0 </pose>
-            <visualize>false</visualize>
-            <update_rate>10</update_rate>
-            <ray>
-                <scan>
-                    <horizontal>
-                        <samples>360</samples>
-                        <min_angle>-3.14</min_angle>
-                        <max_angle>3.14</max_angle>
-                    </horizontal>
-                </scan>
-                <range>
-                    <min>0.15</min>
-                    <max>6.0</max>
-                    <!-- <max>12.0</max> -->
-                    <resolution>0.01500</resolution>
-		        </range>
-                <noise>
-                    <type>gaussian</type>
-                    <mean>0.0</mean>
-                    <stddev>0.01</stddev>
-                </noise>
-            </ray>
-            <plugin name="laser_controller" filename="libgazebo_ros_ray_sensor.so">
-                <ros>
-                    <argument>~/out:=scan</argument>
-                </ros>
-                <output_type>sensor_msgs/LaserScan</output_type>
-                <frame_name>lidar_frame</frame_name>
-            </plugin>
-        </sensor>
-    </gazebo>
-    <gazebo reference="camera_frame">
-        <material>Gazebo/Black</material>
-        <sensor name="camera" type="camera">
-            <pose> camera_radius 0 0 0 0 0 </pose>
-            <visualize>true</visualize>
-            <update_rate>10</update_rate>
-            <camera>
-                <horizontal_fov>1.089</horizontal_fov>
-                <image>
-                    <format>R8G8B8</format>
-                    <width>640</width>
-                    <height>480</height>
-                </image>
-                <clip>
-                    <near>0.05</near>
-                    <far>8.0</far>
-                </clip>
-            </camera>
-            <plugin name="camera_controller" filename="libgazebo_ros_camera.so">
-                <frame_name>camera_optical_frame</frame_name>
-            </plugin>
-        </sensor>
-    </gazebo>
-    <gazebo reference="imu_frame">
-        <material>Gazebo/Blue</material>
-        <gravity>true</gravity>
-        <sensor name="mpu6050_imu" type="imu">
-            <pose> 0 0 0 0 0 0 </pose>
-            <always_on>1</always_on>
-            <visualize>true</visualize>
-            <update_rate>100</update_rate>
-            <plugin name="imu_controller" filename="libgazebo_ros_imu_sensor.so">
-                <topic_name>imu</topic_name>
-                <frame_name>imu_frame</frame_name>
-                <ros>
-                    <remapping>~/out:=imu_broadcaster/imu</remapping>
-                </ros>
-                <initial_orientation_as_reference>false</initial_orientation_as_reference>
-            </plugin>
-            <always_on>true</always_on>
-            <update_rate>100</update_rate>
-            <visualize>true</visualize>
-            <imu>
-            <angular_velocity>
-                <x>
-                <noise type="gaussian">
-                    <mean>0.0</mean>
-                    <stddev>2e-4</stddev>
-                </noise>
-                </x>
-                <y>
-                <noise type="gaussian">
-                    <mean>0.0</mean>
-                    <stddev>2e-4</stddev>
-                </noise>
-                </y>
-                <z>
-                <noise type="gaussian">
-                    <mean>0.0</mean>
-                    <stddev>2e-4</stddev>
-                </noise>
-                </z>
-            </angular_velocity>
-            <linear_acceleration>
-                <x>
-                <noise type="gaussian">
-                    <mean>0.0</mean>
-                    <stddev>1.7e-2</stddev>
-                </noise>
-                </x>
-                <y>
-                <noise type="gaussian">
-                    <mean>0.0</mean>
-                    <stddev>1.7e-2</stddev>
-                </noise>
-                </y>
-                <z>
-                <noise type="gaussian">
-                    <mean>0.0</mean>
-                    <stddev>1.7e-2</stddev>
-                </noise>
-                </z>
-            </linear_acceleration>
-            <orientation>
-                <x>
-                <noise type="gaussian">
-                    <mean>0.0</mean>
-                    <stddev>2e-3</stddev>
-                    </noise>
-                </x>
-                <y>
-                    <noise type="gaussian">
-                    <mean>0.0</mean>
-                    <stddev>2e-3</stddev>
-                    </noise>
-                </y>
-                <z>
-                    <noise type="gaussian">
-                    <mean>0.0</mean>
-                    <stddev>2e-3</stddev>
-                    </noise>
-                </z>
-                </orientation>
-            </imu>
-        </sensor>
-    </gazebo>
 </robot>

File: src/bob_description/urdf/imu.xacro (robot description, xacro)
@@ -26,3 +26,86 @@
         </collision>
     </link>
+    <gazebo reference="imu_frame">
+        <material>Gazebo/Blue</material>
+        <gravity>true</gravity>
+        <sensor name="mpu6050_imu" type="imu">
+            <pose> 0 0 0 0 0 0 </pose>
+            <always_on>1</always_on>
+            <visualize>true</visualize>
+            <update_rate>100</update_rate>
+            <plugin name="imu_controller" filename="libgazebo_ros_imu_sensor.so">
+                <topic_name>imu</topic_name>
+                <frame_name>imu_frame</frame_name>
+                <ros>
+                    <remapping>~/out:=imu_broadcaster/imu</remapping>
+                </ros>
+                <initial_orientation_as_reference>false</initial_orientation_as_reference>
+            </plugin>
+            <always_on>true</always_on>
+            <update_rate>100</update_rate>
+            <visualize>true</visualize>
+            <imu>
+            <angular_velocity>
+                <x>
+                <noise type="gaussian">
+                    <mean>0.0</mean>
+                    <stddev>2e-4</stddev>
+                </noise>
+                </x>
+                <y>
+                <noise type="gaussian">
+                    <mean>0.0</mean>
+                    <stddev>2e-4</stddev>
+                </noise>
+                </y>
+                <z>
+                <noise type="gaussian">
+                    <mean>0.0</mean>
+                    <stddev>2e-4</stddev>
+                </noise>
+                </z>
+            </angular_velocity>
+            <linear_acceleration>
+                <x>
+                <noise type="gaussian">
+                    <mean>0.0</mean>
+                    <stddev>1.7e-2</stddev>
+                </noise>
+                </x>
+                <y>
+                <noise type="gaussian">
+                    <mean>0.0</mean>
+                    <stddev>1.7e-2</stddev>
+                </noise>
+                </y>
+                <z>
+                <noise type="gaussian">
+                    <mean>0.0</mean>
+                    <stddev>1.7e-2</stddev>
+                </noise>
+                </z>
+            </linear_acceleration>
+            <orientation>
+                <x>
+                <noise type="gaussian">
+                    <mean>0.0</mean>
+                    <stddev>2e-3</stddev>
+                    </noise>
+                </x>
+                <y>
+                    <noise type="gaussian">
+                    <mean>0.0</mean>
+                    <stddev>2e-3</stddev>
+                    </noise>
+                </y>
+                <z>
+                    <noise type="gaussian">
+                    <mean>0.0</mean>
+                    <stddev>2e-3</stddev>
+                    </noise>
+                </z>
+                </orientation>
+            </imu>
+        </sensor>
+    </gazebo>
 </robot>

File: src/bob_description/urdf/lidar.xacro (robot description, xacro)
@@ -30,3 +30,38 @@
         </inertial>
     </link>
+    <gazebo reference="lidar_frame">
+        <material>Gazebo/Red</material>
+        <sensor name="lidar" type="ray">
+            <pose> 0 0 0 0 0 0 </pose>
+            <visualize>false</visualize>
+            <update_rate>10</update_rate>
+            <ray>
+                <scan>
+                    <horizontal>
+                        <samples>360</samples>
+                        <min_angle>-3.14</min_angle>
+                        <max_angle>3.14</max_angle>
+                    </horizontal>
+                </scan>
+                <range>
+                    <min>0.15</min>
+                    <max>6.0</max>
+                    <!-- <max>12.0</max> -->
+                    <resolution>0.01500</resolution>
+		        </range>
+                <noise>
+                    <type>gaussian</type>
+                    <mean>0.0</mean>
+                    <stddev>0.01</stddev>
+                </noise>
+            </ray>
+            <plugin name="laser_controller" filename="libgazebo_ros_ray_sensor.so">
+                <ros>
+                    <argument>~/out:=scan</argument>
+                </ros>
+                <output_type>sensor_msgs/LaserScan</output_type>
+                <frame_name>lidar_frame</frame_name>
+            </plugin>
+        </sensor>
+    </gazebo>
 </robot>

Commit message: implement the IMU

File: src/bob_description/ros2_control/bob.ros2_control.xacro (robot description, xacro)
@@ -26,4 +26,24 @@
         <state_interface name="alarm"/>
       </joint>
+    </ros2_control>
+    <!-- MPU6050 sensor-->
+    <ros2_control name='MPU6050' type='sensor'>
+      <hardware>
+        <plugin>bob_bringup/MPU6050Hardware</plugin>
+          <param name='sensor_name'>mpu6050</param>
+          <param name='frame_id'>imu_frame</param>
+      </hardware>
+      <sensor name='mpu6050'>
+        <state_interface name='orientation.x'/>
+        <state_interface name='orientation.y'/>
+        <state_interface name='orientation.z'/>
+        <state_interface name='orientation.w'/>
+        <state_interface name='angular_velocity.x'/>
+        <state_interface name='angular_velocity.y'/>
+        <state_interface name='angular_velocity.z'/>
+        <state_interface name='linear_acceleration.x'/>
+        <state_interface name='linear_acceleration.y'/>
+        <state_interface name='linear_acceleration.z'/>
+      </sensor>
     </ros2_control>
   </xacro:unless>

File: src/bob_description/urdf/imu.xacro (robot description, xacro)
@@ -1,20 +1,20 @@
 <?xml version="1.0"?>
 <robot xmlns:xacro="http://www.ros.org/wiki/xacro" >
-    <xacro:property name="acc_x_dim" value="0.02"/>
-    <xacro:property name="acc_y_dim" value="0.015"/>
-    <xacro:property name="acc_z_dim" value="0.001"/>
-    <xacro:property name="acc_x_offset" value="0.13"/>
-    <xacro:property name="acc_density" value="2710.0"/>
-    <xacro:property name="acc_mass" value="${acc_density*acc_x_dim*acc_y_dim*acc_z_dim}"/>
+    <xacro:property name="imu_x_dim" value="0.02"/>
+    <xacro:property name="imu_y_dim" value="0.015"/>
+    <xacro:property name="imu_z_dim" value="0.001"/>
+    <xacro:property name="imu_x_offset" value="0.13"/>
+    <xacro:property name="imu_density" value="2710.0"/>
+    <xacro:property name="imu_mass" value="${imu_density*imu_x_dim*imu_y_dim*imu_z_dim}"/>
     <!-- LIDAR LINK -->
-	<joint name="acc_joint" type="fixed">
+	<joint name="imu_joint" type="fixed">
         <parent link="chassis"/>
         <child link="imu_frame"/>
-        <origin xyz="${acc_x_offset} 0 ${acc_z_dim*0.5+main_body_z_dim}"/>
+        <origin xyz="${imu_x_offset} 0 ${imu_z_dim*0.5+main_body_z_dim}"/>
     </joint>
     <link name="imu_frame">
         <visual>
             <geometry>
-                <box size="${acc_x_dim} ${acc_y_dim} ${acc_z_dim}"/>
+                <box size="${imu_x_dim} ${imu_y_dim} ${imu_z_dim}"/>
             </geometry>
             <material name="blue"/>
@@ -22,5 +22,5 @@
         <collision>
             <geometry>
-                <box size="${acc_x_dim} ${acc_y_dim} ${acc_z_dim}"/>
+                <box size="${imu_x_dim} ${imu_y_dim} ${imu_z_dim}"/>
             </geometry>
         </collision>
@@ -32,5 +32,5 @@
             <pose> 0 0 0 0 0 0 </pose>
             <always_on>1</always_on>
-            <visualize>true</visualize>
+            <visualize>false</visualize>
             <update_rate>100</update_rate>
             <plugin name="imu_controller" filename="libgazebo_ros_imu_sensor.so">
@@ -44,5 +44,5 @@
             <always_on>true</always_on>
             <update_rate>100</update_rate>
-            <visualize>true</visualize>
+            <visualize>false</visualize>
             <imu>
             <angular_velocity>

File: src/bob_description/urdf/lidar.xacro (robot description, xacro)
@@ -34,5 +34,5 @@
         <sensor name="lidar" type="ray">
             <pose> 0 0 0 0 0 0 </pose>
-            <visualize>false</visualize>
+            <visualize>true</visualize>
             <update_rate>10</update_rate>
             <ray>
@@ -40,6 +40,6 @@
                     <horizontal>
                         <samples>360</samples>
-                        <min_angle>-3.14</min_angle>
-                        <max_angle>3.14</max_angle>
+                        <min_angle>-2.0</min_angle>
+                        <max_angle>2.0</max_angle>
                     </horizontal>
                 </scan>
